File: SDR-RX/SDR-RX.sch (KiCad schematic (older format))
At the start: 52 parts, among them U1 Si4734-D60-GU, Y1 32.768kHz

Commit message: Project & PCB file added
Parts:
- removed R? (x2): 12k, Resistor_SMD:R_0603_1608Metric_Pad0.98x0.95mm_HandSolder, symbol Device:R
- removed RFGND, RFGND? (x8): GND1, symbol power:GND1
- added R3, R4: 10k, Resistor_SMD:R_0603_1608Metric_Pad0.98x0.95mm_HandSolder, symbol Device:R
- FB1: renamed from FB?; footprint Inductor_SMD:L_1206_3216Metric_Pad1.22x1.90mm_HandSolder -> Inductor_SMD:L_1210_3225Metric_Pad1.42x2.65mm_HandSolder; LCSC Part # C94305 -> C124093
- J2: renamed from J?; footprint (none) -> Connector_JST:JST_XH_S2B-XH-A_1x02_P2.50mm_Horizontal
- J5: renamed from J?; footprint (none) -> Connector_PinHeader_2.54mm:PinHeader_1x03_P2.54mm_Vertical
- SW1: renamed from SW?; symbol Switch:SW_MEC_5E -> Switch:SW_DPST_x2
- TP1, TP2, TP3, TP4, TP5: renamed from TP?; footprint (none) -> TestPoint:TestPoint_Pad_D1.5mm
- gave numbers to parts that had none: 30
Connections:
- net labels added: GND1
- wire segments 161 -> 156
- no-connect marks 3 -> 7
Other:
- moved on the sheet: J3

Commit message: changed J2 footprint
Parts:
- J2: footprint Connector_JST:JST_XH_S2B-XH-A_1x02_P2.50mm_Horizontal -> Connector_JST:JST_XH_S2B-XH-A-1_1x02_P2.50mm_Horizontal
Changed lines of the file:
@@
 F 0 "J2" H 4442 1525 50  0000 C CNN
 F 1 "Conn_01x02_Female" H 4442 1616 50  0000 C CNN
-F 2 "Connector_JST:JST_XH_S2B-XH-A_1x02_P2.50mm_Horizontal" H 4550 1850 50  0001 C CNN
+F 2 "Connector_JST:JST_XH_S2B-XH-A-1_1x02_P2.50mm_Horizontal" H 4550 1850 50  0001 C CNN
 F 3 "~" H 4550 1850 50  0001 C CNN
 	1    4550 1850

Commit message: added SW2
Parts:
- added SW2: 3V3 J5/J2, Button_Switch_SMD:SW_SPDT_CK-JS102011SAQN, symbol Switch:SW_SPDT
Connections:
- wire segments 156 -> 163
Other:
- moved on the sheet: C12, C13, C5, C6, D1, D4, F1, FB1, J2, J5, TP5, U3

Commit message: put parts closer on PCB
Parts:
- FB1: value 0Ω @ 100MHZ 1A -> 1kΩ @ 100MHz
- J2: value Conn_01x02_Female -> Vin
- J3: value Conn_Coaxial -> FM Antenna
- J4: value Conn_Coaxial -> AM Antenna
Changed lines of the file:
@@
 P 5150 2550
 F 0 "J2" H 5042 2225 50  0000 C CNN
-F 1 "Conn_01x02_Female" H 5042 2316 50  0000 C CNN
+F 1 "Vin " H 5042 2316 50  0000 C CNN
 F 2 "Connector_JST:JST_XH_S2B-XH-A-1_1x02_P2.50mm_Horizontal" H 5150 2550 50  0001 C CNN
 F 3 "~" H 5150 2550 50  0001 C CNN
@@
 P 6850 2450
 F 0 "FB1" V 6576 2450 50  0000 C CNN
-F 1 "0Ω @ 100MHZ 1A" V 6667 2450 50  0000 C CNN
+F 1 "1kΩ @ 100MHz" V 6667 2450 50  0000 C CNN
 F 2 "Inductor_SMD:L_1210_3225Metric_Pad1.42x2.65mm_HandSolder" V 6780 2450 50  0001 C CNN
 F 3 "https://datasheet.lcsc.com/szlcsc/1811141410_FH-Guangdong-Fenghua-Advanced-Tech-CBG322513U102T_C124093.pdf" H 6850 2450 50  0001 C CNN
@@
 P 6750 5400
 F 0 "J4" H 6850 5375 50  0000 L CNN
-F 1 "Conn_Coaxial" H 6850 5284 50  0000 L CNN
+F 1 "AM Antenna" H 6850 5284 50  0000 L CNN
 F 2 "Connector_Coaxial:SMA_Samtec_SMA-J-P-X-ST-EM1_EdgeMount" H 6750 5400 50  0001 C CNN
 F 3 " ~" H 6750 5400 50  0001 C CNN
@@
 P 6250 6600
 F 0 "J3" H 6350 6575 50  0000 L CNN
-F 1 "Conn_Coaxial" H 6350 6484 50  0000 L CNN
+F 1 "FM Antenna" H 6350 6484 50  0000 L CNN
 F 2 "Connector_Coaxial:SMA_Samtec_SMA-J-P-X-ST-EM1_EdgeMount" H 6250 6600 50  0001 C CNN
 F 3 " ~" H 6250 6600 50  0001 C CNN
